File: PCB/Hambapad.kicad_pcb (KiCad board)
At the start: 2 copper layers, 60.5 x 58.4 mm, 9 parts, among them J2 Conn_01x04_Pin, SW1 SW_Push, SW2 SW_Push, SW3 SW_Push, SW4 SW_Push, SW5 SW_Push, SW6 SW_Push, SW7 RotaryEncoder_Switch, U1 XIAO-RP2040-DIP

Commit message: Add files via upload
Parts:
- added G***: LOGO, New folder:hama, F.Cu at (160.6, 109.9)
